File: LED Driver/LED Driver.kicad_sch (KiCad schematic)
At the start: 33 parts, among them J1 Conn_Coaxial, J2 Conn_01x02_Socket, J3 Screw_Terminal_01x02, J4 Conn_01x02_Socket, U1 SN74LVC2G04MDCKREP, U2 SN74LVC2G04MDCKREP, U3 74LVC2G08DP-Q100H, U4 LM317_SOT-223

Commit message: Added more comments to LED driver
Parts:
- C7: URL (none) -> https://www.digikey.ca/en/products/detail/chemi-con/EKMA500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
- R2: Mfr. # (none) -> RP73PF1J698RBTDF
- U1: URL (none) -> https://www.digikey.ca/en/products/detail/texas-instruments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; Url https://www.digikey.ca/en/products/detail/texas-instruments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 -> (none)
- U4: URL (none) -> https://www.digikey.ca/en/products/detail/texas-instruments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
Other:
- note added: "R4 and R5 can be any value (including 0 ohms)"
- note added: "eTime delay should be approx t = C2*(R3+R2)*1.2 1.2 comes from the 74LVC2G04 has a 0.7*Vcc high level threshold The smallest time possible with this setup is 6.7ns Biggest is 163ns R2 is a low tempco resistor and C2 is NP0"
- note removed: "Time delay should be approx t = C2*(R3+R2)*1.2 1.2 comes from the 74LVC2G04 has a 0.7*Vcc high level threshold The smallest time possible with this setup is 6.7ns Biggest is 163ns"
Changed lines of the file:
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@@
     (fill (type none))
   )
-  (text "Time delay should be approx t = C2*(R3+R2)*1.2\n1.2 comes from the 74LVC2G04 has a 0.7*Vcc high level threshold\n\nThe smallest time possible with this setup is 6.7ns\nBiggest is 163ns\n"
-    (at 92.964 29.083 0)
+  (text "eTime delay should be approx t = C2*(R3+R2)*1.2\n1.2 comes from the 74LVC2G04 has a 0.7*Vcc high level threshold\n\nThe smallest time possible with this setup is 6.7ns\nBiggest is 163ns\n\nR2 is a low tempco resistor and C2 is NP0\n"
+    (at 94.615 29.845 0)
     (effects (font (size 1.27 1.27)) (justify left bottom))
   )
@@
   )
   (text "Expected Input Voltage 12V" (at 16.51 113.03 0)
+    (effects (font (size 1.27 1.27)) (justify left bottom))
+  )
+  (text "R4 and R5 can be any value (including 0 ohms)\n" (at 230.505 36.195 0)
     (effects (font (size 1.27 1.27)) (justify left bottom))
   )
@@
     )
     (property "Datasheet" "~" (at 118.745 40.64 0)
+      (effects (font (size 1.27 1.27)) hide)
+    )
+    (property "Mfr. #" "RP73PF1J698RBTDF" (at 118.745 40.64 0)
       (effects (font (size 1.27 1.27)) hide)
     )
@@
       (effects (font (size 1.27 1.27)) hide)
     )
+    (property "URL" "https://www.digikey.ca/en/products/detail/chemi-con/EKMA500ETD100MF07D/3999919" (at 80.645 123.825 90)
+      (effects (font (size 1.27 1.27)) hide)
+    )
     (pin "1")
     (pin "2")
@@
       (effects (font (size 1.27 1.27)) hide)
     )
-    (property "Url" "https://www.digikey.ca/en/products/detail/texas-instruments/SN74LVC2G04MDCKREP/1628995" (at 85.852 93.726 0)
+    (property "URL" "https://www.digikey.ca/en/products/detail/texas-instruments/SN74LVC2G04MDCKREP/1628995" (at 85.852 93.726 0)
       (effects (font (size 1.27 1.27)) hide)
     )
@@
       (effects (font (size 1.27 1.27)) hide)
     )
-    (property "Url" "https://www.digikey.ca/en/products/detail/texas-instruments/SN74LVC2G04MDCKREP/1628995" (at 122.682 83.185 0)
+    (property "URL" "https://www.digikey.ca/en/products/detail/texas-instruments/SN74LVC2G04MDCKREP/1628995" (at 122.682 83.185 0)
       (effects (font (size 1.27 1.27)) hide)
     )
@@
       (effects (font (size 1.27 1.27)) hide)
     )
-    (property "Url" "https://www.digikey.ca/en/products/detail/texas-instruments/SN74LVC2G04MDCKREP/1628995" (at 85.725 76.962 0)
+    (property "URL" "https://www.digikey.ca/en/products/detail/texas-instruments/SN74LVC2G04MDCKREP/1628995" (at 85.725 76.962 0)
       (effects (font (size 1.27 1.27)) hide)
     )
@@
       (effects (font (size 1.27 1.27)) hide)
     )
+    (property "URL" "https://www.digikey.ca/en/products/detail/texas-instruments/LM317MDCYR/454187" (at 134.62 125.095 0)
+      (effects (font (size 1.27 1.27)) hide)
+    )
